File: schematics/audio_board/audio_board.kicad_sch (KiCad schematic)
At the start: 70 parts, among them J1 pyr ctrl, J2 mic, J3 power, J4 pyr ctrl, J6 pyr in, J7 audio ctrl, J8 speaker, U1 TPS613222ADBV, U2 MCP1802x-xx02xOT, U3 MCP1802x-xx02xOT, U4 TPS613222ADBV, U5 PAM8302AAD, U6 TLV9061xDBV, U7 TLV9061xDBV

Commit message: Placing parts onto PCB...
Parts:
- removed C12, C17, C20: 100n, Capacitor_SMD:C_0603_1608Metric_Pad1.08x0.95mm_HandSolder, symbol Device:C
- removed D4, D5, D6, D7: LED, LED_THT:LED_D5.0mm, symbol Device:LED
- removed R12, R13, R14, R4: 1k, Capacitor_SMD:C_0603_1608Metric_Pad1.08x0.95mm_HandSolder, symbol Device:R
Connections:
- net at U7.3 (+): now also C9.2, R24.2, R32.1
- net at C25.1, R27.2, R28.1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: no longer C9.2, R24.2, R32.1
Other:
- moved on the sheet: C25, C26, C27, J2, R27, R28, R29, R31, U7

Commit message: Correct package for audio amplifier. It is MSOP-8, not SOIC-8.
Parts:
- U5: footprint Package_SO:SOIC-8_3.9x4.9mm_P1.27mm -> Package_SO:MSOP-8_3x3mm_P0.65mm
Changed lines of the file:
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@@
 			)
 		)
-		(property "Footprint" "Package_SO:SOIC-8_3.9x4.9mm_P1.27mm"
+		(property "Footprint" "Package_SO:MSOP-8_3x3mm_P0.65mm"
 			(at 317.5 58.42 0)
 			(effects
