File: schematics/audio_board/power_ctrl.kicad_sch (KiCad schematic)
At the start: 7 parts, among them Q3 NPN, Q4 PMOS

Commit message: Placing footprints.
Parts:
- C15, R10, R8: footprint Capacitor_SMD:C_0603_1608Metric -> Capacitor_SMD:C_0603_1608Metric_Pad1.08x0.95mm_HandSolder
- R20, R9: footprint Resistor_SMD:R_0603_1608Metric -> Resistor_SMD:R_0603_1608Metric_Pad0.98x0.95mm_HandSolder
Changed lines of the file:
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@@
 			)
 		)
-		(property "Footprint" "Capacitor_SMD:C_0603_1608Metric"
+		(property "Footprint" "Capacitor_SMD:C_0603_1608Metric_Pad1.08x0.95mm_HandSolder"
 			(at 148.082 82.55 90)
 			(effects
@@
 			)
 		)
-		(property "Footprint" "Resistor_SMD:R_0603_1608Metric"
+		(property "Footprint" "Resistor_SMD:R_0603_1608Metric_Pad0.98x0.95mm_HandSolder"
 			(at 151.638 68.58 90)
 			(effects
@@
 			)
 		)
-		(property "Footprint" "Capacitor_SMD:C_0603_1608Metric"
+		(property "Footprint" "Capacitor_SMD:C_0603_1608Metric_Pad1.08x0.95mm_HandSolder"
 			(at 134.62 97.028 90)
 			(effects
@@
 			)
 		)
-		(property "Footprint" "Resistor_SMD:R_0603_1608Metric"
+		(property "Footprint" "Resistor_SMD:R_0603_1608Metric_Pad0.98x0.95mm_HandSolder"
 			(at 130.048 102.87 90)
 			(effects
@@
 			)
 		)
-		(property "Footprint" "Capacitor_SMD:C_0603_1608Metric"
+		(property "Footprint" "Capacitor_SMD:C_0603_1608Metric_Pad1.08x0.95mm_HandSolder"
 			(at 173.6852 95.25 0)
 			(effects

Commit message: a
Parts:
- removed Q3: NPN, Package_TO_SOT_SMD:SOT-23, symbol Simulation_SPICE:NPN
- removed Q4: PMOS, Package_TO_SOT_SMD:SOT-23, symbol Simulation_SPICE:PMOS
- added Q1: bc847, Package_TO_SOT_SMD:SOT-23, symbol bc847:bc847
- added Q7: dgm2305ux, Package_TO_SOT_SMD:SOT-23, symbol dgm2305ux:dgm2305ux
Connections:
- net GND: now also Q1.2 (E)
- net pwr: now also Q7.3 (D)
- net pwr_out: now also Q7.2 (S)
- net at R10.2: now also Q1.3 (C)
- net at R8.2: now also Q1.1 (B)
- net at R10.1, R9.2: now also Q7.1 (G)
