File: schematics/audio_board/audio_board.kicad_pcb (KiCad board)
At the start: 2 copper layers, 66 parts, among them J1 servo ctrl, J2 charge en, J3 power, J4 pyr ctrl, J5 servo out, J6 pyr in, J7 Conn_01x06, J8 speaker, Q1 NPN, Q2 PMOS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

Commit message: a
Parts:
- removed Q4, Q6: PMOS, Package_TO_SOT_SMD:SOT-23
- removed Q5: NPN, Package_TO_SOT_SMD:SOT-23
- added Q7: dgm2305ux, Package_TO_SOT_SMD:SOT-23, F.Cu at (80.7, 65.2)
- added Q8: dgm2305ux, Package_TO_SOT_SMD:SOT-23, F.Cu at (91.9, 47.3)
- added Q9: dgm2305ux, Package_TO_SOT_SMD:SOT-23, F.Cu at (91.5, 29.8)
- added R23: 100k, Resistor_SMD:R_0603_1608Metric_Pad0.98x0.95mm_HandSolder, F.Cu at (123.3, 87.2)
- added R24: 100k, Resistor_SMD:R_0603_1608Metric_Pad0.98x0.95mm_HandSolder, F.Cu at (123.3, 90.0)
- added R25: 100k, Resistor_SMD:R_0603_1608Metric_Pad0.98x0.95mm_HandSolder, F.Cu at (123.2, 92.3)
- Q1, Q3: value NPN -> bc847
- Q2: value PMOS -> bc847
- R1: value 2k -> 100k
- moved Q3 39.2 mm to (86.9, 29.7)
- moved R13 32.0 mm to (91.4, 26.9), turned to 180 degrees
- moved R6 31.6 mm to (91.9, 44.4), turned to 180 degrees
- moved C14 30.7 mm to (91.8, 49.9)
- moved C16 30.3 mm to (91.4, 32.6)
- moved R14 29.6 mm to (87.8, 26.9), turned to 180 degrees
- moved R11 28.6 mm to (87.9, 44.4)
- moved R22 25.9 mm to (83.8, 29.7), turned to -90 degrees
- moved R21 24.6 mm to (83.8, 47.3), turned to -90 degrees
- moved R12 24.1 mm to (83.9, 26.9)
- moved R5 23.3 mm to (83.9, 44.4)
- moved Q2 22.4 mm to (87.4, 47.4)
Connections:
- Q1 pad 1: Net-(Q1-C) -> Net-(Q1-B)
- Q1 pad 2: Net-(Q1-B) -> GND
- Q1 pad 3: GND -> Net-(Q1-C)
- Q2 pad 1: /Power ctrl PYR/pwr_out -> Net-(Q2-B)
- Q2 pad 2: Net-(Q2-G) -> GND
- Q2 pad 3: /Vin -> Net-(Q2-C)
- Q3 pad 1: Net-(Q3-C) -> Net-(Q3-B)
- Q3 pad 2: Net-(Q3-B) -> GND
- Q3 pad 3: GND -> Net-(Q3-C)
- R1 pad 1: GND -> /charge_en
- R1 pad 2: /charge_en -> GND
- R10 pad 2: Net-(Q3-C) -> Net-(Q1-C)
- R11 pad 1: Net-(Q2-G) -> Net-(Q8-G)
- R11 pad 2: Net-(Q1-C) -> Net-(Q2-C)
- R12 pad 2: Net-(Q5-B) -> Net-(Q3-B)
- R14 pad 2: Net-(Q5-C) -> Net-(Q3-C)
- R5 pad 2: Net-(Q1-B) -> Net-(Q2-B)
- R6 pad 2: Net-(Q2-G) -> Net-(Q8-G)
- R8 pad 2: Net-(Q3-B) -> Net-(Q1-B)

Commit message: a
Parts:
- removed J2: charge en, Connector_PinSocket_2.54mm:PinSocket_1x01_P2.54mm_Vertical
- removed TP1: +, Connector_Pin:Pin_D1.4mm_L8.5mm_W2.8mm_FlatFork
- removed TP2: -, Connector_Pin:Pin_D1.4mm_L8.5mm_W2.8mm_FlatFork
- added D3: 1N5819, Diode_THT:D_DO-41_SOD81_P7.62mm_Horizontal, F.Cu at (77.5, 96.0)
- added J10: charge en, Connector_PinSocket_2.54mm:PinSocket_1x02_P2.54mm_Vertical, F.Cu at (53.0, 93.2)
- added J9: battery, Connector_PinSocket_2.54mm:PinSocket_1x02_P2.54mm_Vertical, F.Cu at (97.0, 83.5)
- J7: value Conn_01x06 -> audio ctrl
- moved J1 124.0 mm to (53.0, 80.0)
- moved R7 123.5 mm to (59.1, 84.0)
- moved J6 105.2 mm to (97.0, 61.5)
- moved J5 104.5 mm to (97.0, 71.5)
- moved R17 99.4 mm to (57.0, 73.1)
- moved R98 99.4 mm to (59.0, 73.1)
- moved J4 98.5 mm to (53.0, 70.1)
- moved C4 75.0 mm to (65.4, 81.8)
- moved C5 75.0 mm to (76.5, 81.1)
- moved C9 75.0 mm to (74.5, 81.1)
- moved L2 75.0 mm to (65.4, 79.2)
- moved U3 75.0 mm to (71.0, 81.2)
- moved R23 72.4 mm to (57.4, 57.2)
- moved R24 72.1 mm to (57.4, 60.8)
- moved R25 71.5 mm to (57.4, 64.2)
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Connections:
- net Net-(U2-BCLK) renamed /bclk
- D2 pad 2: /power -> /pwr+
- J3 pad 1: /power -> /pwr+
- R2 pad 2: Net-(U2-DIN) -> /lrclk
- R4 pad 2: Net-(U2-LRCLK) -> /din
- U2 pad 1: Net-(U2-DIN) -> /din
- U2 pad 14: Net-(U2-LRCLK) -> /lrclk

Commit message: a
Parts:
- removed C16: 22u, Capacitor_SMD:C_0603_1608Metric_Pad1.08x0.95mm_HandSolder
- removed C3: 100n, Capacitor_SMD:C_0603_1608Metric_Pad1.08x0.95mm_HandSolder
- removed Q3: bc847, Package_TO_SOT_SMD:SOT-23
- removed Q9: dgm2305ux, Package_TO_SOT_SMD:SOT-23
- removed R15, R16, R18, R19, R22, R23, R24, R25: 100k, Resistor_SMD:R_0603_1608Metric_Pad0.98x0.95mm_HandSolder
- removed U2: MAX98357A, Package_DFN_QFN:TQFN-16-1EP_3x3mm_P0.5mm_EP1.23x1.23mm
- added C13: 100n, Capacitor_SMD:C_0603_1608Metric_Pad1.08x0.95mm_HandSolder, F.Cu at (79.9, 58.2)
- added C18: 100n, Capacitor_SMD:C_0603_1608Metric_Pad1.08x0.95mm_HandSolder, F.Cu at (79.9, 56.0)
- added C19: 22u, Capacitor_SMD:C_0603_1608Metric_Pad1.08x0.95mm_HandSolder, F.Cu at (93.8, 56.1)
- added C20: 100n, Capacitor_SMD:C_0603_1608Metric_Pad1.08x0.95mm_HandSolder, F.Cu at (91.8, 56.1)
- added D4: LED, LED_THT:LED_D5.0mm, F.Cu at (64.5, 56.2)
- added D5: LED, LED_THT:LED_D5.0mm, F.Cu at (84.8, 65.0)
- added D6: LED, LED_THT:LED_D5.0mm, F.Cu at (74.0, 86.5)
- added D7: LED, LED_THT:LED_D5.0mm, F.Cu at (90.7, 75.0)
- added R26: 100k, Resistor_SMD:R_0603_1608Metric_Pad0.98x0.95mm_HandSolder, F.Cu at (80.1, 52.5)
- added U5: PAM8302AAD, Package_SO:SOIC-8_3.9x4.9mm_P1.27mm, F.Cu at (86.3, 56.1)
- C2: value 22u -> 100n
- J7: footprint Connector_PinSocket_2.54mm:PinSocket_1x06_P2.54mm_Vertical -> Connector_PinSocket_2.54mm:PinSocket_1x03_P2.54mm_Vertical
- R13: value 100k -> 1k; footprint Resistor_SMD:R_0603_1608Metric_Pad0.98x0.95mm_HandSolder -> Capacitor_SMD:C_0603_1608Metric_Pad1.08x0.95mm_HandSolder
- R2, R4: value 33 -> 1k; footprint Resistor_SMD:R_0603_1608Metric_Pad0.98x0.95mm_HandSolder -> Capacitor_SMD:C_0603_1608Metric_Pad1.08x0.95mm_HandSolder
- R3: value 33 -> 100k
- moved R13 35.3 mm to (69.6, 86.4), turned to 0 degrees
- moved R12 34.4 mm to (89.4, 65.1), turned to 180 degrees
- moved R14 34.0 mm to (86.3, 74.9), turned to 0 degrees
- moved R2 18.7 mm to (75.6, 55.0)
- moved R4 15.1 mm to (68.9, 56.2), turned to 180 degrees
- moved C2 14.3 mm to (76.5, 58.1), turned to -90 degrees
- moved C6 12.9 mm to (66.3, 67.3)
- moved C1 12.9 mm to (76.8, 65.1)
- moved C17 12.9 mm to (74.8, 65.1)
- moved L1 12.9 mm to (66.3, 64.3)
- moved U1 12.9 mm to (71.2, 65.2)
- moved C8 12.9 mm to (59.1, 91.9), turned to 90 degrees
- moved R1 10.8 mm to (60.1, 89.0), turned to 180 degrees
- moved D2 9.25 mm to (69.9, 96.8)
- moved D3 8.72 mm to (69.6, 92.2)
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Connections:
- C2 pad 1: /5V_audio -> /audio_in
- C6 pad 1: /Power ctrl PYR1/pwr_out -> /Vin
- J7 pad 2: Net-(J7-Pin_2) -> GND
- J7 pad 3: Net-(J7-Pin_3) -> /audio_dac
- L1 pad 1: /Power ctrl PYR1/pwr_out -> /Vin
- R12 pad 1: /audio_en -> GND
- R13 pad 1: /Vin -> GND
- R13 pad 2: Net-(Q9-G) -> Net-(D6-K)
- R14 pad 1: Net-(Q9-G) -> GND
- R2 pad 1: Net-(J7-Pin_2) -> /audio_dac
- R2 pad 2: /lrclk -> /audio_in
- R3 pad 1: Net-(J7-Pin_3) -> GND
- R3 pad 2: /bclk -> /audio_dac
- R4 pad 1: Net-(J7-Pin_4) -> GND
- R4 pad 2: /din -> Net-(D4-K)
Routing:
- net GND: track 0.00 -> 320.8 mm, vias 0 -> 13
- net /Vin: track 0.00 -> 78.2 mm, vias 0 -> 4
- net /Vbatt: track 0.00 -> 58.9 mm
- net /pyr_in: track 0.00 -> 48.2 mm, vias 0 -> 2
- net Net-(J5-Pin_3): track 0.00 -> 43.8 mm, vias 0 -> 2
- net /5V_servo: track 0.00 -> 36.6 mm
- net /audio_en: track 0.00 -> 34.7 mm
- net /5V_audio: track 0.00 -> 32.7 mm, vias 0 -> 1
- net /Power ctrl/en: track 0.00 -> 30.4 mm
- net /5V_pyr: track 0.00 -> 25.6 mm, vias 0 -> 1
- net /pwr+: track 0.00 -> 24.6 mm
- net /audio_dac: track 0.00 -> 23.8 mm
- net /Power ctrl/pwr_out: track 0.00 -> 15.1 mm, vias 0 -> 1
- net /charge_en: track 0.00 -> 15.1 mm
- net /pyr_en: track 0.00 -> 14.2 mm
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Other:
- board outline added: 50 x 50 mm

Commit message: a
Parts:
- moved L2 0.81 mm to (65.5, 80.0)
- moved C4 0.70 mm to (65.5, 82.5)
Routing:
- net GND: track 320.8 -> 338.4 mm
- net /5V_audio: track 32.7 -> 43.7 mm
- net /Vin: track 78.2 -> 87.3 mm
- net /Vbatt: track 58.9 -> 61.1 mm
- net /5V_pyr: track 25.6 -> 27.6 mm
- added copper zone on B.Cu, net GND
- added copper zone on F.Cu, net GND

Commit message: I believe, it is finished.
Routing:
- net /Vbatt: track 61.1 -> 56.2 mm
Changed lines of the file:
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@@
 			)
 		)
-		(property "Datasheet" "~"
+		(property "Datasheet" ""
 			(at 0 0 0)
 			(layer "F.Fab")
@@
 			)
 		)
-		(property "Datasheet" "~"
+		(property "Datasheet" ""
 			(at 0 0 0)
 			(layer "F.Fab")
@@
 			)
 		)
-		(property "Datasheet" "~"
+		(property "Datasheet" ""
 			(at 0 0 0)
 			(layer "F.Fab")
@@
 			)
 		)
-		(property "Datasheet" "~"
+		(property "Datasheet" ""
 			(at 0 0 0)
 			(layer "F.Fab")
@@
 			)
 		)
-		(property "Datasheet" "~"
+		(property "Datasheet" ""
 			(at 0 0 0)
 			(layer "F.Fab")
@@
 			)
 		)
-		(property "Datasheet" "~"
+		(property "Datasheet" ""
 			(at 0 0 90)
 			(layer "F.Fab")
@@
 			)
 		)
-		(property "Datasheet" "~"
+		(property "Datasheet" ""
 			(at 0 0 90)
 			(layer "F.Fab")
@@
 			)
 		)
-		(property "Datasheet" "~"
+		(property "Datasheet" ""
 			(at 0 0 90)
 			(layer "F.Fab")
@@
 			)
 		)
-		(property "Datasheet" "~"
+		(property "Datasheet" ""
 			(at 0 0 0)
 			(layer "F.Fab")
@@
 			)
 		)
-		(property "Datasheet" "~"
+		(property "Datasheet" ""
 			(at 0 0 0)
 			(layer "F.Fab")
@@
 			)
 		)
-		(property "URL" "https://www.digikey.com/en/products/detail/yageo/AC0603JR-072K2L/5896418"
-			(at 0 0 180)
-			(unlocked yes)
-			(layer "F.Fab")
-			(hide yes)
-			(effects
-				(font
-					(size 1 1)
-					(thickness 0.15)
-				)
-			)
-		)
 		(property ki_fp_filters "R_*")
 		(sheetname "/")
@@
 			)
 		)
-		(property "Datasheet" "~"
+		(property "Datasheet" ""
 			(at 0 0 0)
 			(layer "F.Fab")
@@
 			)
 		)
-		(property "Datasheet" "~"
+		(property "Datasheet" ""
 			(at 0 0 0)
 			(layer "F.Fab")
@@
 			)
 		)
-		(property "Datasheet" "~"
+		(property "Datasheet" ""
 			(at 0 0 90)
 			(layer "F.Fab")
@@
 			)
 		)
-		(property "Datasheet" "~"
+		(property "Datasheet" ""
 			(at 0 0 90)
 			(layer "F.Fab")
@@
 			)
 		)
-		(property "Datasheet" "~"
+		(property "Datasheet" ""
 			(at 0 0 90)
 			(layer "F.Fab")
@@
 			)
 		)
-		(property "Datasheet" "~"
+		(property "Datasheet" ""
 			(at 0 0 0)
 			(layer "F.Fab")
@@
 			)
 		)
-		(property "Datasheet" "~"
+		(property "Datasheet" ""
 			(at 0 0 0)
 			(layer "F.Fab")
@@
 			)
 		)
-		(property "Datasheet" "~"
+		(property "Datasheet" ""
 			(at 0 0 90)
 			(layer "F.Fab")
@@
 			)
 		)
-		(property "Datasheet" "~"
+		(property "Datasheet" ""
 			(at 0 0 0)
 			(layer "F.Fab")
@@
 			)
 		)
-		(property "Datasheet" "~"
+		(property "Datasheet" ""
 			(at 0 0 0)
 			(layer "F.Fab")
@@
 			)
 		)
-		(property "Datasheet" "~"
+		(property "Datasheet" ""
 			(at 0 0 0)
 			(layer "F.Fab")
@@
 			)
 		)
-		(property "Datasheet" "~"
+		(property "Datasheet" ""
 			(at 0 0 90)
 			(layer "F.Fab")
@@
 			)
 		)
-		(property "Datasheet" "~"
+		(property "Datasheet" ""
 			(at 0 0 90)
 			(layer "F.Fab")
@@
 			)
 		)
-		(property "Datasheet" "~"
+		(property "Datasheet" ""
 			(at 0 0 0)
 			(layer "F.Fab")
@@
 			)
 		)
-		(property "Datasheet" "~"
+		(property "Datasheet" ""
 			(at 0 0 0)
 			(layer "F.Fab")
@@
 			)
 		)
-		(property "Datasheet" "~"
+		(property "Datasheet" ""
 			(at 0 0 90)
 			(layer "F.Fab")
@@
 			)
 		)
-		(property "Datasheet" "~"
+		(property "Datasheet" ""
 			(at 0 0 0)
 			(layer "F.Fab")
@@
 			)
 		)
-		(property "Datasheet" "~"
+		(property "Datasheet" ""
 			(at 0 0 0)
 			(layer "F.Fab")
@@
 			)
 		)
-		(property "Datasheet" "~"
+		(property "Datasheet" ""
 			(at 0 0 0)
 			(layer "F.Fab")
@@
 			)
 		)
-		(property "Datasheet" "~"
+		(property "Datasheet" ""
 			(at 0 0 0)
 			(layer "F.Fab")
@@
 			)
 		)
-		(property "Datasheet" "~"
+		(property "Datasheet" ""
 			(at 0 0 90)
 			(layer "F.Fab")
@@
 			)
 		)
-		(property "Datasheet" "~"
+		(property "Datasheet" ""
 			(at 0 0 0)
 			(layer "F.Fab")
@@
 			)
 		)
-		(property "Datasheet" "~"
+		(property "Datasheet" ""
 			(at 0 0 0)
 			(layer "F.Fab")
@@
 			)
 		)
-		(property "Datasheet" "~"
+		(property "Datasheet" ""
 			(at 0 0 0)
 			(layer "F.Fab")
@@
 			)
 		)
-		(property "Datasheet" "~"
+		(property "Datasheet" ""
 			(at 0 0 0)
 			(layer "F.Fab")
@@
 			)
 		)
-		(property "Datasheet" "~"
+		(property "Datasheet" ""
 			(at 0 0 90)
 			(layer "F.Fab")
@@
 			)
 		)
-		(property "Datasheet" "~"
+		(property "Datasheet" ""
 			(at 0 0 0)
 			(layer "F.Fab")
@@
 			)
 		)
-		(property "Datasheet" "~"
+		(property "Datasheet" ""
 			(at 0 0 0)
 			(layer "F.Fab")
@@
 			)
 		)
-		(property "Datasheet" "~"
+		(property "Datasheet" ""
 			(at 0 0 0)
 			(layer "F.Fab")
@@
 			)
 		)
-		(property "Datasheet" "~"
+		(property "Datasheet" ""
 			(at 0 0 0)
 			(layer "F.Fab")
@@
 			)
 		)
-		(property "Datasheet" "~"
+		(property "Datasheet" ""
 			(at 0 0 0)
 			(layer "F.Fab")
@@
 			)
 		)
-		(property "Datasheet" "~"
+		(property "Datasheet" ""
 			(at 0 0 0)
 			(layer "F.Fab")
@@
 			)
 		)
-		(property "Datasheet" "~"
+		(property "Datasheet" ""
 			(at 0 0 0)
 			(layer "F.Fab")
@@
 			)
 		)
-		(property "Datasheet" "~"
+		(property "Datasheet" ""
 			(at 0 0 0)
 			(layer "F.Fab")
@@
 			)
 		)
-		(property "Datasheet" "~"
+		(property "Datasheet" ""
 			(at 0 0 0)
 			(layer "F.Fab")
@@
 			)
 		)
-		(property "Datasheet" "~"
+		(property "Datasheet" ""
 			(at 0 0 0)
 			(layer "F.Fab")
@@
 			)
 		)
-		(property "Datasheet" "~"
+		(property "Datasheet" ""
 			(at 0 0 0)
 			(layer "F.Fab")
@@
 			)
 		)
-		(property "Datasheet" "~"
+		(property "Datasheet" ""
 			(at 0 0 0)
 			(layer "F.Fab")
@@
 			)
 		)
-		(property "Datasheet" "~"
+		(property "Datasheet" ""
 			(at 0 0 90)
 			(layer "F.Fab")
@@
 			)
 		)
-		(property "Datasheet" "~"
+		(property "Datasheet" ""
 			(at 0 0 0)
 			(layer "F.Fab")
@@
 			)
 		)
-		(property "Datasheet" "~"
+		(property "Datasheet" ""
 			(at 0 0 90)
 			(layer "F.Fab")
@@
 			)
 		)
-		(property "Datasheet" "~"
+		(property "Datasheet" ""
 			(at 0 0 0)
 			(layer "F.Fab")
@@
 			)
 		)
-		(property "Datasheet" "~"
+		(property "Datasheet" ""
 			(at 0 0 90)
 			(layer "F.Fab")
@@
 			)
 		)
-		(property "Datasheet" "~"
+		(property "Datasheet" ""
 			(at 0 0 0)
 			(layer "F.Fab")
@@
 			)
 		)
-		(property "Datasheet" "~"
+		(property "Datasheet" ""
 			(at 0 0 90)
 			(layer "F.Fab")
@@
 			)
 		)
-		(property "Datasheet" "~"
+		(property "Datasheet" ""
 			(at 0 0 0)
 			(layer "F.Fab")
@@
 			)
 		)
-		(property "Datasheet" "~"
+		(property "Datasheet" ""
 			(at 0 0 0)
 			(layer "F.Fab")
@@
 	)
 	(segment
-		(start 97 83.46)
-		(end 93.5 86.96)
-		(width 0.4)
-		(layer "F.Cu")
-		(net 6)
-	)
-	(segment
 		(start 58.19 96.75)
 		(end 58.19 93.71)
@@
 		(min_thickness 0.25)
 		(filled_areas_thickness no)
-		(fill
+		(fill yes
 			(thermal_gap 0.5)
 			(thermal_bridge_width 0.5)
