File: schematics/mp_board/mp_board.kicad_sch (KiCad schematic)
At the start: 34 parts, among them J10 swd, J11 stm_boot, J17 rst_mcu, J6 MY_USB_B, J9 uart1, U1 MCP1802x-xx02xOT, Y1 Crystal

Commit message: a
Parts:
- added C2: 4u7, Capacitor_SMD:C_0603_1608Metric, symbol Device:C
- added R10, R5, R6, R7, R8, R9: 10k, Resistor_SMD:R_0603_1608Metric, symbol Device:R
- added R11, R12, R13, R14: 33, Resistor_SMD:R_0603_1608Metric_Pad0.98x0.95mm_HandSolder, symbol Device:R
- added R3, R4: 22, symbol Device:R
- added U2: W25Q128JVS, Package_SO:SOIC-8_5.3x5.3mm_P1.27mm, symbol Memory_Flash:W25Q128JVS
Connections:
- net GND: now also C2.2, U2.4 (GND)
- net VDD: now also C2.1, R10.1, R5.1, R6.1, R7.1, R8.1, R9.1, U2.8 (VCC)
- net led-0: now also U10.50 (PA15___JTDI); no longer U10.21 (PA5)
- net led-1: now also U10.51 (PC10___USART4_TX); no longer U10.22 (PA6)
- net led-2: now also U10.52 (PC11__USART4_RX); no longer U10.23 (PA7)
- net led-3: now also U10.53 (PC12)
- net usb_d+: now also R3.2; no longer J6.3 (D+)
- net usb_d-: now also R4.2; no longer J6.2 (D-)
- net spi2_miso: now reaches U10.10 (PC2)
- net spi2_miso: now also R14.1
- net spi2_mosi: now reaches U10.11 (PC3)
- net spi2_mosi: now also R13.1
- net spi2_sck: now reaches U10.34 (PB13)
- net spi2_sck: now also R12.1
- net batt_charge_en renamed flash_cs_pin
- net flash_cs_pin: now also R11.1
- net batt_sense: no longer names the net of U10.14 (PA0-WKUP)
- net scl_host_a renamed i2c1_sck
- net i2c1_sck: now also R5.2
- net scl_host_b renamed i2c2_sck
- net i2c2_sck: now also R7.2
- net scl_host_c: no longer names the net of U10.41 (PA8__OTG_FS_SOF)
- net sda_host_a renamed i2c1_sda
- net i2c1_sda: now also R6.2
- net sda_host_b renamed i2c2_sda
- net i2c2_sda: now also R8.2
- net sda_host_c: no longer names the net of U10.40 (PC9)
- net stm_rx: no longer names the net of U10.17 (PA3)
- net stm_tx: no longer names the net of U10.16 (PA2)
- new net: J6.2 (D-), R4.1
- new net: J6.3 (D+), R3.1
- new net flash_cs: R11.2, U2.1 (~{CS})
- new net flash_di: R13.2, U2.5 (DI/IO_{0})
- new net flash_do: R14.2, U2.2 (DO/IO_{1})
- new net flash_hold: R9.2, U2.7 (~{HOLD}/~{RESET}/IO_{3})
- new net flash_sck: R12.2, U2.6 (CLK)
- new net flash_wp: R10.2, U2.3 (~{WP}/IO_{2})
- no-connect marks 32 -> 24
Other:
- moved on the sheet: C23, C24, C27, C28, C29, C30, C31, C4, C9, D1, D3, D4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

Commit message: Coarsly finished the scheme. Assigned footprints. Have concerns about flash chip SOIC8 size though.
Parts:
- removed D1, D4: LED, LED_THT:LED_D3.0mm, symbol Device:LED
- removed D2: 1N5819, Diode_THT:D_DO-41_SOD81_P7.62mm_Horizontal, symbol Device:D_Schottky
- removed R2, R92: 1k, Resistor_SMD:R_0603_1608Metric, symbol Device:R
- added J1: i2c_1, Connector_PinHeader_2.54mm:PinHeader_1x04_P2.54mm_Vertical, symbol Connector:Conn_01x04_Pin
- added J2: i2c_2, Connector_PinHeader_2.54mm:PinHeader_1x04_P2.54mm_Vertical, symbol Connector:Conn_01x04_Pin
- added J3: pins_b, Connector_PinSocket_2.54mm:PinSocket_2x09_P2.54mm_Vertical, symbol Connector_Generic:Conn_02x09_Counter_Clockwise
- added J4: power_a, Connector_PinSocket_2.54mm:PinSocket_2x03_P2.54mm_Vertical, symbol Connector_Generic:Conn_02x03_Counter_Clockwise
- added J7: power_b, Connector_PinSocket_2.54mm:PinSocket_2x03_P2.54mm_Vertical, symbol Connector_Generic:Conn_02x03_Counter_Clockwise
- added J8: pins_a, Connector_PinSocket_2.54mm:PinSocket_2x09_P2.54mm_Vertical, symbol Connector_Generic:Conn_02x09_Counter_Clockwise
- R3, R4: footprint (none) -> Resistor_SMD:R_0603_1608Metric
Connections:
- net Vin is gone; now on net Vbus: C5.1, U1.1 (VIN), U1.3 (~{SHDN})
- net GND: now also J9.2 (Pin_2), J1.2 (Pin_2), J2.2 (Pin_2), J3.10 (Pin_10), J4.2 (Pin_2), J4.5 (Pin_5), J7.2 (Pin_2), J7.5 (Pin_5), J8.10 (Pin_10); no longer J9.4 (Pin_4)
- net VDD: now also J9.4 (Pin_4), J1.4 (Pin_4), J2.4 (Pin_4), J4.1 (Pin_1), J4.6 (Pin_6), J7.1 (Pin_1), J7.6 (Pin_6); no longer J9.3 (Pin_3)
- net Vbus: now also J4.3 (Pin_3), J4.4 (Pin_4), J7.3 (Pin_3), J7.4 (Pin_4)
- net i2c1_sck: now also J1.1 (Pin_1)
- net i2c1_sda: now also J1.3 (Pin_3)
- net i2c2_sck: now also J2.1 (Pin_1)
- net i2c2_sda: now also J2.3 (Pin_3)
- net led-0: now also J3.3 (Pin_3)
- net led-1: now also J3.15 (Pin_15)
- net uart1-tx: now also J9.3 (Pin_3); no longer J9.2 (Pin_2)
- net pa0: now reaches U10.14 (PA0-WKUP)
- net pa0: now also J8.1 (Pin_1)
- net pa1: now reaches U10.15 (PA1)
- net pa1: now also J8.2 (Pin_2)
- net pa2: now reaches U10.16 (PA2)
- net pa2: now also J8.3 (Pin_3)
- net pa3: now reaches U10.17 (PA3)
- net pa3: now also J8.4 (Pin_4)
- net pc13: now reaches U10.2 (PC13-TAMPER-RTC)
- net pc13: now also J3.12 (Pin_12)
- net pa4: now reaches U10.20 (PA4)
- net pa4: now also J8.5 (Pin_5)
- net pa5: now reaches U10.21 (PA5)
- net pa5: now also J8.6 (Pin_6)
- net pa6: now reaches U10.22 (PA6)
- net pa6: now also J8.7 (Pin_7)
- net pa7: now reaches U10.23 (PA7)
- net pa7: now also J8.8 (Pin_8)
- net pc4: now reaches U10.24 (PC4)
- net pc4: now also J3.6 (Pin_6)
- net pc5: now reaches U10.25 (PC5)
- net pc5: now also J3.7 (Pin_7)
- net pb0: now reaches U10.26 (PB0)
- net pb0: now also J8.17 (Pin_17)
- net pb1: now reaches U10.27 (PB1)
- net pb1: now also J8.16 (Pin_16)
- net pb14: now reaches U10.35 (PB14___OTG_HS_DM)
- net pb14: now also J3.1 (Pin_1)
- net pb15: now reaches U10.36 (PB15___OTG_HS_DP)
- net pb15: now also J3.2 (Pin_2)
- net pc6: now reaches U10.37 (PC6__USART6_TX)
- net pc6: now also J3.8 (Pin_8)
- net pc7: now reaches U10.38 (PC7___USART6_RX)
- net pc7: now also J3.18 (Pin_18)
- net pc8: now reaches U10.39 (PC8)
- net pc8: now also J3.17 (Pin_17)
- net pc9: now reaches U10.40 (PC9)
- net pc9: now also J3.16 (Pin_16)
- net pa8: now reaches U10.41 (PA8__OTG_FS_SOF)
- net pa8: now also J8.18 (Pin_18)
- net pd2: now reaches U10.54 (PD2)
- net pd2: now also J3.11 (Pin_11)
- net pb3: now reaches U10.55 (PB3)
- net pb3: now also J8.15 (Pin_15)
- net pb4: now reaches U10.56 (PB4)
- net pb4: now also J8.14 (Pin_14)
- net pb5: now reaches U10.57 (PB5)
- net pb5: now also J8.13 (Pin_13)
- net pb8: now reaches U10.61 (PB8)
- net pb8: now also J8.11 (Pin_11)
- net pb9: now reaches U10.62 (PB9)
- net pb9: now also J8.12 (Pin_12)
- net pc0: now reaches U10.8 (PC0)
- net pc0: now also J3.4 (Pin_4)
- net pc1: now reaches U10.9 (PC1)
- net pc1: now also J3.5 (Pin_5)
- net pc14: now reaches U10.3 (PC14-OSC32_IN)
- net pc14: now also J8.9 (Pin_9)
- net pc15: now reaches U10.4 (PC15-OSC32_OUT)
- net pc15: now also J3.9 (Pin_9)
- net led-2 renamed pc11
- net pc11: now also J3.14 (Pin_14)
- net led-3 renamed pc12
- net pc12: now also J3.13 (Pin_13)
- no-connect marks 24 -> 3
Other:
- moved on the sheet: R5, R6, R7, R8

Commit message: Made tripple sockets. Mid pins are all ground for shielding.
Parts:
- removed J11: stm_boot, Connector_PinHeader_2.54mm:PinHeader_1x02_P2.54mm_Vertical, symbol Connector:Conn_01x02_Pin
- removed J17: rst_mcu, Connector_PinHeader_2.54mm:PinHeader_1x02_P2.54mm_Vertical, symbol Connector:Conn_01x02_Pin
- removed J3: pins_b, Connector_PinSocket_2.54mm:PinSocket_2x09_P2.54mm_Vertical, symbol Connector_Generic:Conn_02x09_Counter_Clockwise
- removed J4: power_a, Connector_PinSocket_2.54mm:PinSocket_2x03_P2.54mm_Vertical, symbol Connector_Generic:Conn_02x03_Counter_Clockwise
- removed J7: power_b, Connector_PinSocket_2.54mm:PinSocket_2x03_P2.54mm_Vertical, symbol Connector_Generic:Conn_02x03_Counter_Clockwise
- removed J8: pins_a, Connector_PinSocket_2.54mm:PinSocket_2x09_P2.54mm_Vertical, symbol Connector_Generic:Conn_02x09_Counter_Clockwise
- added J12: pins_e, Connector_PinHeader_2.54mm:PinHeader_1x12_P2.54mm_Vertical, symbol Connector_Generic:Conn_01x12
- added J13: pins_f, Connector_PinHeader_2.54mm:PinHeader_1x12_P2.54mm_Vertical, symbol Connector_Generic:Conn_01x12
- added J3: boot_rst, Connector_PinHeader_2.54mm:PinHeader_1x04_P2.54mm_Vertical, symbol Connector:Conn_01x04_Pin
- added J4: pins_b, Connector_PinHeader_2.54mm:PinHeader_1x12_P2.54mm_Vertical, symbol Connector_Generic:Conn_01x12
- added J5: pins_a, Connector_PinHeader_2.54mm:PinHeader_1x12_P2.54mm_Vertical, symbol Connector_Generic:Conn_01x12
- added J7: pins_c, Connector_PinHeader_2.54mm:PinHeader_1x12_P2.54mm_Vertical, symbol Connector_Generic:Conn_01x12
- added J8: pins_d, Connector_PinHeader_2.54mm:PinHeader_1x12_P2.54mm_Vertical, symbol Connector_Generic:Conn_01x12
Connections:
- net GND: now also J12.1 (Pin_1), J12.10 (Pin_10), J12.11 (Pin_11), J12.12 (Pin_12), J12.2 (Pin_2), J12.3 (Pin_3), J12.4 (Pin_4), J12.5 (Pin_5), J12.6 (Pin_6), J12.7 (Pin_7), J12.8 (Pin_8), J12.9 (Pin_9), J13.12 (Pin_12), J13.2 (Pin_2), J3.2 (Pin_2), J4.1 (Pin_1), J4.10 (Pin_10), J4.11 (Pin_11), J4.12 (Pin_12), J4.2 (Pin_2), J4.3 (Pin_3), J4.4 (Pin_4), J4.5 (Pin_5), J4.6 (Pin_6), J4.7 (Pin_7), J4.8 (Pin_8), J4.9 (Pin_9), J5.2 (Pin_2), J7.12 (Pin_12), J7.2 (Pin_2), J8.2 (Pin_2)
- net VDD: now also J13.3 (Pin_3), J3.4 (Pin_4), J5.3 (Pin_3), J7.3 (Pin_3), J8.3 (Pin_3)
- net Vbus: now also J13.1 (Pin_1), J5.1 (Pin_1), J7.1 (Pin_1), J8.1 (Pin_1)
- net boot0: now also J3.3 (Pin_3)
- net led-0: now also J8.6 (Pin_6)
- net led-1: now also J13.7 (Pin_7)
- net pa0: now also J5.4 (Pin_4)
- net pa1: now also J5.5 (Pin_5)
- net pa2: now also J5.6 (Pin_6)
- net pa3: now also J5.7 (Pin_7)
- net pa4: now also J5.8 (Pin_8)
- net pa5: now also J5.9 (Pin_9)
- net pa6: now also J5.10 (Pin_10)
- net pa7: now also J5.11 (Pin_11)
- net pa8: now also J7.4 (Pin_4)
- net pb0: now also J7.5 (Pin_5)
- net pb1: now also J7.6 (Pin_6)
- net pb14: now also J8.4 (Pin_4)
- net pb15: now also J8.5 (Pin_5)
- net pb3: now also J7.7 (Pin_7)
- net pb4: now also J7.8 (Pin_8)
- net pb5: now also J7.9 (Pin_9)
- net pb8: now also J7.11 (Pin_11)
- net pb9: now also J7.10 (Pin_10)
- net pc0: now also J8.7 (Pin_7)
- net pc1: now also J8.8 (Pin_8)
- net pc11: now also J13.8 (Pin_8)
- net pc12: now also J13.9 (Pin_9)
- net pc13: now also J13.10 (Pin_10)
- net pc14: now also J5.12 (Pin_12)
- net pc15: now also J8.12 (Pin_12)
- net pc4: now also J8.9 (Pin_9)
- net pc5: now also J8.10 (Pin_10)
- net pc6: now also J8.11 (Pin_11)
- net pc7: now also J13.4 (Pin_4)
- net pc8: now also J13.5 (Pin_5)
- net pc9: now also J13.6 (Pin_6)
- net pd2: now also J13.11 (Pin_11)
- net rst_mcu: now also J3.1 (Pin_1)
- no-connect marks 3 -> 2
Other:
- moved on the sheet: R87

Commit message: Wiring.
Connections:
- net pa0: now also J8.5 (Pin_5); no longer J5.4 (Pin_4)
- net pa1: now also J13.6 (Pin_6); no longer J5.5 (Pin_5)
- net pa2: now also J13.8 (Pin_8); no longer J5.6 (Pin_6)
- net pa3: now also J13.11 (Pin_11); no longer J5.7 (Pin_7)
- net pa4: now also J13.9 (Pin_9); no longer J5.8 (Pin_8)
- net pa5: now also J13.10 (Pin_10); no longer J5.9 (Pin_9)
- net pa6: now also J8.12 (Pin_12); no longer J5.10 (Pin_10)
- net pa7: now also J8.7 (Pin_7); no longer J5.11 (Pin_11)
- net pa8: now also J7.6 (Pin_6); no longer J7.4 (Pin_4)
- net pb0: now also J13.5 (Pin_5); no longer J7.5 (Pin_5)
- net pb1: now also J8.11 (Pin_11); no longer J7.6 (Pin_6)
- net pb15: now also J13.4 (Pin_4); no longer J8.5 (Pin_5)
- net pb3: now also J7.8 (Pin_8); no longer J7.7 (Pin_7)
- net pb4: now also J5.8 (Pin_8); no longer J7.8 (Pin_8)
- net pb8: now also J5.9 (Pin_9); no longer J7.11 (Pin_11)
- net pc0: now also J5.12 (Pin_12); no longer J8.7 (Pin_7)
- net pc11: now also J5.6 (Pin_6); no longer J13.8 (Pin_8)
- net pc12: now also J7.7 (Pin_7); no longer J13.9 (Pin_9)
- net pc13: now also J5.10 (Pin_10); no longer J13.10 (Pin_10)
- net pc14: now also J7.11 (Pin_11); no longer J5.12 (Pin_12)
- net pc15: now also J5.11 (Pin_11); no longer J8.12 (Pin_12)
- net pc6: now also J7.4 (Pin_4); no longer J8.11 (Pin_11)
- net pc7: now also J5.4 (Pin_4); no longer J13.4 (Pin_4)
- net pc8: now also J7.5 (Pin_5); no longer J13.5 (Pin_5)
- net pc9: now also J5.5 (Pin_5); no longer J13.6 (Pin_6)
- net pd2: now also J5.7 (Pin_7); no longer J13.11 (Pin_11)
Changed lines of the file:
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@@
 	)
 	(label "pd2"
-		(at 472.44 280.67 180)
+		(at 302.26 270.51 180)
 		(effects
 			(font
@@
 	)
 	(label "pc12"
-		(at 472.44 275.59 180)
+		(at 369.57 270.51 180)
 		(effects
 			(font
@@
 	)
 	(label "pb1"
-		(at 369.57 267.97 180)
+		(at 412.75 280.67 180)
 		(effects
 			(font
@@
 	)
 	(label "pa8"
-		(at 369.57 262.89 180)
+		(at 369.57 267.97 180)
 		(effects
 			(font
@@
 	)
 	(label "pa3"
-		(at 302.26 270.51 180)
+		(at 472.44 280.67 180)
 		(effects
 			(font
@@
 	)
 	(label "pa0"
-		(at 302.26 262.89 180)
+		(at 412.75 265.43 180)
 		(effects
 			(font
@@
 	)
 	(label "pa6"
-		(at 302.26 278.13 180)
+		(at 412.75 283.21 180)
 		(effects
 			(font
@@
 	)
 	(label "pa1"
-		(at 302.26 265.43 180)
+		(at 472.44 267.97 180)
 		(effects
 			(font
@@
 	)
 	(label "pb4"
-		(at 369.57 273.05 180)
+		(at 302.26 273.05 180)
 		(effects
 			(font
@@
 	)
 	(label "pa4"
-		(at 302.26 273.05 180)
+		(at 472.44 275.59 180)
 		(effects
 			(font
@@
 	)
 	(label "pa5"
-		(at 302.26 275.59 180)
+		(at 472.44 278.13 180)
 		(effects
 			(font
@@
 	)
 	(label "pc11"
-		(at 472.44 273.05 180)
+		(at 302.26 267.97 180)
 		(effects
 			(font
@@
 	)
 	(label "pc0"
-		(at 412.75 270.51 180)
+		(at 302.26 283.21 180)
 		(effects
 			(font
@@
 	)
 	(label "pc15"
-		(at 412.75 283.21 180)
+		(at 302.26 280.67 180)
 		(effects
 			(font
@@
 	)
 	(label "pb8"
-		(at 369.57 280.67 180)
+		(at 302.26 275.59 180)
 		(effects
 			(font
@@
 	)
 	(label "pa7"
-		(at 302.26 280.67 180)
+		(at 412.75 270.51 180)
 		(effects
 			(font
@@
 	)
 	(label "pb15"
-		(at 412.75 265.43 180)
+		(at 472.44 262.89 180)
 		(effects
 			(font
@@
 	)
 	(label "pa2"
-		(at 302.26 267.97 180)
+		(at 472.44 273.05 180)
 		(effects
 			(font
@@
 	)
 	(label "pc9"
-		(at 472.44 267.97 180)
+		(at 302.26 265.43 180)
 		(effects
 			(font
@@
 	)
 	(label "pb3"
-		(at 369.57 270.51 180)
+		(at 369.57 273.05 180)
 		(effects
 			(font
@@
 	)
 	(label "pc7"
-		(at 472.44 262.89 180)
+		(at 302.26 262.89 180)
 		(effects
 			(font
@@
 	)
 	(label "pc6"
-		(at 412.75 280.67 180)
+		(at 369.57 262.89 180)
 		(effects
 			(font
@@
 	)
 	(label "pc8"
-		(at 472.44 265.43 180)
+		(at 369.57 265.43 180)
 		(effects
 			(font
@@
 	)
 	(label "pc14"
-		(at 302.26 283.21 180)
+		(at 369.57 280.67 180)
 		(effects
 			(font
@@
 	)
 	(label "pc13"
-		(at 472.44 278.13 180)
+		(at 302.26 278.13 180)
 		(effects
 			(font
@@
 	)
 	(label "pb0"
-		(at 369.57 265.43 180)
-		(effects
-			(font
+		(at 472.44 265.43 180)
+		(effects
+			(font

Commit message: Wiring.
Connections:
- net led-0: now also J5.5 (Pin_5); no longer J8.6 (Pin_6)
- net led-1: now also J7.6 (Pin_6); no longer J13.7 (Pin_7)
- net pa0: now also J8.11 (Pin_11); no longer J8.5 (Pin_5)
- net pa1: now also J13.11 (Pin_11); no longer J13.6 (Pin_6)
- net pa2: now also J8.10 (Pin_10); no longer J13.8 (Pin_8)
- net pa3: now also J13.10 (Pin_10); no longer J13.11 (Pin_11)
- net pa4: now also J8.9 (Pin_9); no longer J13.9 (Pin_9)
- net pa5: now also J13.9 (Pin_9); no longer J13.10 (Pin_10)
- net pa6: now also J8.8 (Pin_8); no longer J8.12 (Pin_12)
- net pa7: now also J13.8 (Pin_8); no longer J8.7 (Pin_7)
- net pa8: now also J7.5 (Pin_5); no longer J7.6 (Pin_6)
- net pb0: now also J8.6 (Pin_6); no longer J13.5 (Pin_5)
- net pb1: now also J13.6 (Pin_6); no longer J8.11 (Pin_11)
- net pb14: now also J13.5 (Pin_5); no longer J8.4 (Pin_4)
- net pb15: now also J8.5 (Pin_5); no longer J13.4 (Pin_4)
- net pc1: now also J8.12 (Pin_12); no longer J8.8 (Pin_8)
- net pc4: now also J8.7 (Pin_7); no longer J8.9 (Pin_9)
- net pc5: now also J13.7 (Pin_7); no longer J8.10 (Pin_10)
- net pc6: now also J13.4 (Pin_4); no longer J7.4 (Pin_4)
- net pc7: now also J8.4 (Pin_4); no longer J5.4 (Pin_4)
- net pc8: now also J7.4 (Pin_4); no longer J7.5 (Pin_5)
- net pc9: now also J5.4 (Pin_4); no longer J5.5 (Pin_5)
Changed lines of the file:
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@@
 	)
 	(label "pc1"
-		(at 412.75 273.05 180)
+		(at 412.75 283.21 180)
 		(effects
 			(font
@@
 	)
 	(label "led-0"
-		(at 412.75 267.97 180)
+		(at 302.26 265.43 180)
 		(effects
 			(font
@@
 	)
 	(label "pb1"
-		(at 412.75 280.67 180)
+		(at 472.44 267.97 180)
 		(effects
 			(font
@@
 	)
 	(label "pa8"
-		(at 369.57 267.97 180)
+		(at 369.57 265.43 180)
 		(effects
 			(font
@@
 	)
 	(label "pa3"
-		(at 472.44 280.67 180)
+		(at 472.44 278.13 180)
 		(effects
 			(font
@@
 	)
 	(label "pc4"
-		(at 412.75 275.59 180)
+		(at 412.75 270.51 180)
 		(effects
 			(font
@@
 	)
 	(label "pa0"
-		(at 412.75 265.43 180)
+		(at 412.75 280.67 180)
 		(effects
 			(font
@@
 	)
 	(label "pa6"
-		(at 412.75 283.21 180)
+		(at 412.75 273.05 180)
 		(effects
 			(font
@@
 	)
 	(label "pa1"
-		(at 472.44 267.97 180)
+		(at 472.44 280.67 180)
 		(effects
 			(font
@@
 	)
 	(label "pb14"
-		(at 412.75 262.89 180)
+		(at 472.44 265.43 180)
 		(effects
 			(font
@@
 	)
 	(label "pa4"
-		(at 472.44 275.59 180)
+		(at 412.75 275.59 180)
 		(effects
 			(font
@@
 	)
 	(label "pa5"
-		(at 472.44 278.13 180)
+		(at 472.44 275.59 180)
 		(effects
 			(font
@@
 	)
 	(label "pa7"
-		(at 412.75 270.51 180)
+		(at 472.44 273.05 180)
 		(effects
 			(font
@@
 	)
 	(label "pb15"
-		(at 472.44 262.89 180)
+		(at 412.75 265.43 180)
 		(effects
 			(font
@@
 	)
 	(label "pa2"
-		(at 472.44 273.05 180)
+		(at 412.75 278.13 180)
 		(effects
 			(font
@@
 	)
 	(label "pc9"
-		(at 302.26 265.43 180)
+		(at 302.26 262.89 180)
 		(effects
 			(font
@@
 	)
 	(label "pc7"
-		(at 302.26 262.89 180)
+		(at 412.75 262.89 180)
 		(effects
 			(font
@@
 	)
 	(label "pc6"
+		(at 472.44 262.89 180)
+		(effects
+			(font
+				(size 1.27 1.27)
+			)
+			(justify right bottom)
+		)
+	)
+	(label "pc8"
 		(at 369.57 262.89 180)
 		(effects
@@
 		)
 	)
-	(label "pc8"
-		(at 369.57 265.43 180)
-		(effects
-			(font
-				(size 1.27 1.27)
-			)
-			(justify right bottom)
-		)
-	)
 	(label "led-1"
-		(at 472.44 270.51 180)
+		(at 369.57 267.97 180)
 		(effects
 			(font
@@
 	)
 	(label "pb0"
-		(at 472.44 265.43 180)
+		(at 412.75 267.97 180)
 		(effects
 			(font
@@
 	)
 	(label "pc5"
-		(at 412.75 278.13 180)
-		(effects
-			(font
+		(at 472.44 270.51 180)
+		(effects
+			(font
