File: schematics/override_board/override_board/override_board.kicad_pcb (KiCad board)
At the start: 2 copper layers, 35 parts, among them J1 Conn_02x05_Counter_Clockwise, J2 Conn_02x06_Counter_Clockwise, U3 TLV9061xDBV, U4 TLV9061xDBV

Commit message: I feel, the override board is done.
Parts:
- removed J2: Conn_02x06_Counter_Clockwise, Connector_PinHeader_2.54mm:PinHeader_2x06_P2.54mm_Vertical
- added J3: Conn_02x05_Odd_Even, Connector_PinHeader_2.54mm:PinHeader_2x05_P2.54mm_Vertical, F.Cu at (78.2, 91.9)
- J1: value Conn_02x05_Counter_Clockwise -> Conn_02x06_Odd_Even; footprint Connector_PinHeader_2.54mm:PinHeader_2x05_P2.54mm_Vertical -> Connector_PinHeader_2.54mm:PinHeader_2x06_P2.54mm_Vertical
- moved C4 57.4 mm to (102.1, 106.2), turned to -90 degrees
- moved C8 56.8 mm to (89.2, 94.1), turned to -90 degrees
- moved C7 56.3 mm to (85.9, 93.9)
- moved R6 55.6 mm to (85.1, 95.4)
- moved U2 53.1 mm to (92.3, 94.5), turned to 90 degrees
- moved C13 52.1 mm to (100.6, 93.2)
- moved R3 50.4 mm to (101.1, 103.6), turned to 180 degrees
- moved R7 49.8 mm to (96.3, 94.5), turned to 0 degrees
- moved R4 49.6 mm to (100.1, 106.2), turned to 90 degrees
- moved U3 49.3 mm to (97.0, 105.5), turned to 90 degrees
- moved C5 49.1 mm to (93.9, 105.3), turned to -90 degrees
- moved C9 48.5 mm to (96.3, 96.3), turned to 180 degrees
- moved R13 47.0 mm to (100.6, 89.7), turned to 180 degrees
- moved R8 46.9 mm to (99.8, 95.0), turned to 180 degrees
- moved R14 46.4 mm to (100.6, 91.4), turned to 180 degrees
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Connections:
- J1 pad 1: GND -> /V_batt_out
- J1 pad 10: /V_batt_in -> GND
- J1 pad 3: GND -> /en_in
- J1 pad 5: GND -> VDD
- J1 pad 6: /pot_y_out -> GND
- J1 pad 7: /pot_x_out -> /L2_out
- J1 pad 8: /L2_in -> GND
- J1 pad 9: /V_pot_rail -> /pot_x_in
Routing:
- net GND: track 0.00 -> 181.3 mm, vias 0 -> 26
- net VDD: track 0.00 -> 58.8 mm, vias 0 -> 5
- net /en: track 0.00 -> 34.5 mm, vias 0 -> 3
- net /V_batt_out: track 0.00 -> 16.5 mm
- net Net-(U3--): track 0.00 -> 15.9 mm
- net Net-(U4--): track 0.00 -> 15.2 mm
- net /V_batt_in: track 0.00 -> 15.0 mm, vias 0 -> 3
- net /L2_out: track 0.00 -> 12.0 mm
- net Net-(U1-on): track 0.00 -> 10.9 mm
- net Net-(U2-no): track 0.00 -> 7.62 mm
- net Net-(U5-com): track 0.00 -> 7.09 mm
- net Net-(U4-+): track 0.00 -> 6.94 mm
- net Net-(U3-+): track 0.00 -> 6.50 mm
- net /en_in: track 0.00 -> 5.41 mm
- net /V_pot_rail: track 0.00 -> 5.03 mm
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- added copper zone on B.Cu, net GND
- added copper zone on F.Cu, net GND
- added copper zone on In1.Cu, net GND
- added copper zone on In2.Cu, net GND
Other:
- board outline added: 33.5 x 22 mm
- copper layers 2 -> 4
